File: toads_breakout.kicad_pcb (KiCad board)
At the start: 2 copper layers, 30 x 40 mm, 9 parts, among them J1 Conn_02x06_Odd_Even, J2 Conn_01x05, Q1 NPN

Commit message: v1.1
Parts:
- added D2: PTT, LED_SMD:LED_0805_2012Metric, F.Cu at (130.6, 126.1)
- added D3: POW, LED_SMD:LED_0805_2012Metric, F.Cu at (130.6, 119.3)
- added D4: COS, LED_SMD:LED_0805_2012Metric, F.Cu at (130.6, 122.7)
- added H1: MountingHole, MountingHole:MountingHole_2.5mm_Pad, F.Cu at (130.2, 97.6)
- added H2: MountingHole, MountingHole:MountingHole_2.5mm_Pad, F.Cu at (154.2, 97.6)
- added H3: MountingHole, MountingHole:MountingHole_2.5mm_Pad, F.Cu at (130.2, 131.6)
- added H4: MountingHole, MountingHole:MountingHole_2.5mm_Pad, F.Cu at (154.2, 131.6)
- added R2: 1K, Resistor_SMD:R_0805_2012Metric_Pad1.20x1.40mm_HandSolder, F.Cu at (134.1, 122.7)
- added R3: 1K, Resistor_SMD:R_0805_2012Metric_Pad1.20x1.40mm_HandSolder, F.Cu at (134.1, 119.3)
- added R4: 1K, Resistor_SMD:R_0805_2012Metric_Pad1.20x1.40mm_HandSolder, F.Cu at (134.1, 126.1)
- added SW1: SW_SPDT, Matt:SW-SPDT-C49023767, F.Cu at (155.3, 106.8)
- added U1: MSW_Logo, Matt:MSW, B.Cu at (148.3, 106.7)
- J2: footprint Connector_PinHeader_2.54mm:PinHeader_1x05_P2.54mm_Vertical -> Connector_PinHeader_2.54mm:PinHeader_1x06_P2.54mm_Vertical
- moved D1 27.7 mm to (147.2, 104.4)
- moved R1 12.0 mm to (144.0, 105.0)
- moved Q1 7.99 mm to (145.9, 108.8)
- moved C2 7.88 mm to (139.8, 122.0), turned to 0 degrees
- moved C1 5.63 mm to (139.8, 124.0), turned to 0 degrees
- moved J2 1.27 mm to (135.8, 131.6)
Connections:
- J1 pad 1: unconnected-(J1-Pin_1-Pad1) -> +5V
- J2 pad 2: PTT -> VREF
- J2 pad 3: AUD_RX -> PTT
- J2 pad 4: AUD_TX -> AUD_RX
- J2 pad 5: COS -> AUD_TX
- RV2 pad 1: AFL -> GND
- RV2 pad 3: GND -> Net-(SW1-B)
Routing:
- net COS: track 7.33 -> 48.2 mm, vias 0 -> 1
- net VOL_DN: track 37.4 -> 7.70 mm
- net +3V3: track 0.00 -> 24.8 mm
- net GPI03: track 12.0 -> 36.2 mm, vias 0 -> 2
- net AFR: track 0.00 -> 23.7 mm, vias 0 -> 1
- net PTT: track 46.2 -> 24.5 mm
- net Net-(SW1-B): track 0.00 -> 11.2 mm, vias 0 -> 1
- net Net-(C1-Pad2): track 11.7 -> 2.50 mm
- net Net-(C2-Pad2): track 23.1 -> 16.4 mm
- net MIC: track 27.2 -> 29.7 mm, vias 0 -> 2
- net AFL: track 16.5 -> 18.7 mm, vias 0 -> 1
- net Net-(D4-A): track 0.00 -> 1.60 mm
- net Net-(D3-A): track 0.00 -> 1.60 mm
- net Net-(D2-A): track 0.00 -> 1.60 mm
- net AUD_TX: track 13.1 -> 12.6 mm, vias 0 -> 1
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Other:
- board text added: "L"
- board text added: "NC"
- board text added: "R"
- board text removed: "+"

Commit message: Bump to v1.1 - not released yet
Parts:
- J2: value Conn_01x05 -> Conn_01x06
- moved D1 23.2 mm to (150.3, 81.4)
- moved R2 23.2 mm to (137.2, 99.7)
- moved D4 23.2 mm to (133.6, 99.7)
- moved U1 23.2 mm to (151.4, 83.7)
- moved C1 23.2 mm to (142.8, 101.1)
- moved C2 23.2 mm to (142.8, 99.1)
- moved H1 23.2 mm to (133.3, 74.6)
- moved H2 23.2 mm to (157.3, 74.6)
- moved H3 23.2 mm to (133.3, 108.6)
- moved H4 23.2 mm to (157.3, 108.6)
- moved J1 23.2 mm to (139.3, 73.6)
- moved J2 23.2 mm to (138.9, 108.6)
- moved R3 23.2 mm to (137.2, 96.3)
- moved R4 23.2 mm to (137.2, 103.1)
- moved RV1 23.2 mm to (153.3, 98.3)
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