File: toads_breakout.kicad_sch (KiCad schematic)
At the start: 9 parts, among them J1 Conn_02x06_Odd_Even, J2 Conn_01x05, Q1 NPN

Commit message: v1.1
Parts:
- removed Q1: NPN, Package_TO_SOT_SMD:SOT-23_Handsoldering, symbol Transistor_BJT:BC547
- added D2: PTT, LED_SMD:LED_0805_2012Metric, symbol Device:LED_Small
- added D3: POW, LED_SMD:LED_0805_2012Metric, symbol Device:LED_Small
- added D4: COS, LED_SMD:LED_0805_2012Metric, symbol Device:LED_Small
- added H1, H2, H3, H4: MountingHole, MountingHole:MountingHole_2.5mm_Pad, symbol Mechanical:MountingHole
- added Q1: NPN, Package_TO_SOT_SMD:SOT-23_Handsoldering, symbol Matt:NPN-C2145
- added R2, R3, R4: 1K, Resistor_SMD:R_0805_2012Metric_Pad1.20x1.40mm_HandSolder, symbol Device:R_Small_US
- added SW1: SW_SPDT, Matt:SW-SPDT-C49023767, symbol Switch:SW_SPDT
- added U1: MSW_Logo, Matt:MSW, symbol Matt:MSW_Logo
- J1: LCSC# (none) -> C124388
- J2: value Conn_01x05 -> Conn_01x06; footprint Connector_PinHeader_2.54mm:PinHeader_1x05_P2.54mm_Vertical -> Connector_PinHeader_2.54mm:PinHeader_1x06_P2.54mm_Vertical; symbol Connector_Generic:Conn_01x05 -> Connector_Generic:Conn_01x06; LCSC# (none) -> C37208
Connections:
- net +3V3: now also R3.1
- net +5V: now also J1.1 (Pin_1)
- net AFL: now also SW1.1 (A); no longer RV2.1
- net AFR: now also SW1.3 (C)
- net AUD_RX: now also J2.4 (Pin_4); no longer J2.3 (Pin_3)
- net AUD_TX: now also J2.5 (Pin_5); no longer J2.4 (Pin_4)
- net COS: now also J2.6 (Pin_6), R2.1; no longer J2.5 (Pin_5)
- net GND: now also RV2.1, D2.1 (K), D3.1 (K), D4.1 (K), Q1.3 (E); no longer RV2.3
- net GPI03: now also R4.1
- net PTT: now also J2.3 (Pin_3), Q1.1 (C); no longer J2.2 (Pin_2)
- net at R1.2: now also Q1.2 (B)
- new net: D2.2 (A), R4.2
- new net: D4.2 (A), R2.2
- new net: D3.2 (A), R3.2
- new net: RV2.3, SW1.2 (B)
- new net VREF: J2.2 (Pin_2)
- no-connect marks 0 -> 4
Other:
- note added: "Active LOW PTT. Signal on GPI03 triggers Q1 and pulls the PTT line low."
- note added: "Audio from radio through a volume knob to the MIC pin on the TOADS board C1 to block any DC stray voltages (if polarised, + on radio side)"
- note added: "Audio from the left channel of the TOADS board through a volume knob to the radio for transmitting C2 to block any DC stray voltages (if polarised, + on toads side)"
- note added: "COS = Carrior Operated Squelch Diode is to ensure the TOADS board recieves squelch from radio but cannot feed information to the squelch pin Note: It's highly recommended that this be active high logic signalling."
- note added: "V1.1 Release 2025-02-17 DONE: LED on PTT ABANDONED: Switch COS to active high/low radios DONE: Holes in PCB to line up with TOADS board DONE: LED for power indication DONE: Switch to choose audio from AFL or AFR DONE: LED for radio PTT feedback DONE: TX Volume pot the wrong way (clockwise lowers output) DONE: Add LED for COS (GPIO 4) DONE: Transistor pads in wrong place on pcb!!!!!!!! DONE: Add m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"
- note removed: "COS = Carrior Operated Squelch"
- moved on the sheet: C1, C2, D1, J1, R1, RV1, RV2

Commit message: Bump to v1.1 - not released yet
Other:
- note added: "Audio from the left (or right) channel of the TOADS board through a volume knob to the radio for transmitting C2 to block any DC stray voltages (if polarised, + on toads side)"
- note added: "V1.2 Release xxxx-xx-xx DONE: Fix copyright for 2026 DONE: Fix some left/right audio comments"
- note removed: "Audio from the left channel of the TOADS board through a volume knob to the radio for transmitting C2 to block any DC stray voltages (if polarised, + on toads side)"
- moved on the sheet: D1, D2, D4, Q1, R1, R2, R4
